File: hardware/PGTN002.brd (EAGLE design)
At the start: 39.7 x 49.5 mm, 31 parts, among them J1 DCJ0202DCJ0202

Commit message: Fixed MISO and SCK connection between ATTINY44 and ISP10 socket swapped
Connections:
- net N$10: now also IC1.8, R3.1; no longer IC1.9, R2.1
- net N$11: now also IC1.9, R2.1; no longer IC1.8, R3.1
Routing:
- net N$11: track 46.9 -> 50.4 mm
- net N$10: track 48.3 -> 45.7 mm
Other:
- board text added: "PGTN002_2"
- board text removed: "PGTN002_1"
Changed lines of the file:
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@@
 <text x="39.37" y="17.145" size="1.27" layer="25" font="vector">pigatron</text>
 <text x="42.545" y="15.875" size="0.6096" layer="25" font="vector">INDUSTRIES</text>
-<text x="39.37" y="13.97" size="0.8128" layer="25" font="vector">PGTN002_1</text>
+<text x="39.37" y="13.97" size="0.8128" layer="25" font="vector">PGTN002_2</text>
 </plain>
 <attributes>
@@
 </signal>
 <signal name="N$10">
-<contactref element="IC1" pad="9"/>
-<contactref element="R2" pad="1"/>
 <contactref element="MISO" pad="1"/>
-<wire x1="59.69" y1="27.305" x2="62.865" y2="24.13" width="0.3048" layer="1"/>
-<wire x1="59.69" y1="57.15" x2="59.69" y2="27.305" width="0.3048" layer="1"/>
-<wire x1="58.42" y1="58.42" x2="59.69" y2="57.15" width="0.3048" layer="1"/>
-<wire x1="61.595" y1="17.145" x2="59.69" y2="15.24" width="0.3048" layer="1"/>
-<wire x1="61.595" y1="18.415" x2="61.595" y2="17.145" width="0.3048" layer="1"/>
-<wire x1="63.5" y1="20.32" x2="61.595" y2="18.415" width="0.3048" layer="1"/>
-<wire x1="64.135" y1="20.32" x2="63.5" y2="20.32" width="0.3048" layer="1"/>
-<wire x1="64.77" y1="20.955" x2="64.135" y2="20.32" width="0.3048" layer="1"/>
-<wire x1="64.77" y1="22.225" x2="64.77" y2="20.955" width="0.3048" layer="1"/>
-<wire x1="62.865" y1="24.13" x2="64.77" y2="22.225" width="0.3048" layer="1"/>
-</signal>
-<signal name="N$11">
 <contactref element="IC1" pad="8"/>
 <contactref element="R3" pad="1"/>
+<wire x1="59.69" y1="15.24" x2="61.595" y2="17.145" width="0.3048" layer="1"/>
+<wire x1="61.595" y1="17.145" x2="61.595" y2="20.32" width="0.3048" layer="1"/>
+<wire x1="61.595" y1="20.32" x2="62.865" y2="21.59" width="0.3048" layer="1"/>
+<wire x1="62.865" y1="21.59" x2="59.69" y2="21.59" width="0.3048" layer="1"/>
+<wire x1="59.69" y1="21.59" x2="58.42" y2="22.86" width="0.3048" layer="1"/>
+<wire x1="58.42" y1="22.86" x2="58.42" y2="55.88" width="0.3048" layer="1"/>
+</signal>
+<signal name="N$11">
 <contactref element="SCK" pad="1"/>
-<wire x1="61.595" y1="21.59" x2="62.865" y2="21.59" width="0.3048" layer="1"/>
-<wire x1="58.42" y1="18.415" x2="61.595" y2="21.59" width="0.3048" layer="1"/>
-<wire x1="58.42" y1="16.51" x2="58.42" y2="18.415" width="0.3048" layer="1"/>
-<wire x1="57.15" y1="15.24" x2="58.42" y2="16.51" width="0.3048" layer="1"/>
-<wire x1="58.42" y1="18.415" x2="58.42" y2="55.88" width="0.3048" layer="1"/>
+<contactref element="R2" pad="1"/>
+<contactref element="IC1" pad="9"/>
+<wire x1="62.865" y1="24.13" x2="60.96" y2="24.13" width="0.3048" layer="1"/>
+<wire x1="60.96" y1="24.13" x2="59.69" y2="25.4" width="0.3048" layer="1"/>
+<wire x1="59.69" y1="25.4" x2="59.69" y2="57.15" width="0.3048" layer="1"/>
+<wire x1="59.69" y1="57.15" x2="58.42" y2="58.42" width="0.3048" layer="1"/>
+<wire x1="57.15" y1="15.24" x2="58.42" y2="16.51" width="0.3048" layer="16"/>
+<wire x1="58.42" y1="16.51" x2="58.42" y2="22.86" width="0.3048" layer="16"/>
+<wire x1="58.42" y1="22.86" x2="59.69" y2="24.13" width="0.3048" layer="16"/>
+<wire x1="59.69" y1="24.13" x2="62.865" y2="24.13" width="0.3048" layer="16"/>
 </signal>
 <signal name="N$12">
